Commit message: URDF initial standarization

File: tiago_dual_description/robots/tiago_dual.urdf.xacro (robot description, xacro)
@@ -12,41 +12,62 @@
   limitations under the License.
  -->
-<robot  xmlns:xacro="http://ros.org/wiki/xacro"
-        name="tiago_dual" >
-    <xacro:arg name="arm_left" default="tiago-arm"/> <!-- tiago-arm, no-arm -->
-    <xacro:arg name="arm_right" default="tiago-arm"/> <!-- tiago-arm, no-arm -->
-    <xacro:arg name="wrist_model_left" default="wrist-2010"/>
-    <xacro:arg name="wrist_model_right" default="wrist-2010"/>
-    <xacro:arg name="end_effector_left" default="pal-gripper"/> <!-- no-end-effector, pal-gripper, pal-hey5, custom-->
-    <xacro:arg name="end_effector_right" default="pal-gripper"/> <!-- no-end-effector, pal-gripper, pal-hey5, custom-->
-    <xacro:arg name="ft_sensor_left" default="schunk-ft"/> <!--no-ft-sensor, schunk-ft -->
-    <xacro:arg name="ft_sensor_right" default="schunk-ft"/> <!--no-ft-sensor, schunk-ft -->
-    <xacro:arg name="laser_model" default="sick-571"/> <!-- no-laser, hokuyo, sick-551, sick-561, sick-571-->
-    <xacro:arg name="camera_model" default="orbbec-astra"/> <!-- no-camera, orbbec-astra, orbbec-astra-pro, asus-xtion -->
-    <xacro:arg name="has_screen" default="false"/> <!-- true, false -->
-    <xacro:arg name="multiple" default="false"/>
-    <xacro:arg name="base_type" default="pmb2"/> <!-- pmb2, omni_base -->
-    <xacro:arg name="description_calibration_dir" default="$(find tiago_dual_description)/urdf/calibration"/>
-    <xacro:arg name="extrinsic_calibration_dir" default="$(find tiago_dual_description)/urdf/calibration"/>
-    <xacro:arg name="namespace" default=""/>
-    <xacro:arg name="no_safety_eps" default="false"/>
-    <xacro:arg name="use_sim" default="false"/>
-    <xacro:property name="arm_left" value="$(arg arm_left)"/>
-    <xacro:property name="arm_right" value="$(arg arm_right)"/>
-    <xacro:property name="wrist_model_left" value="$(arg wrist_model_left)" />
-    <xacro:property name="wrist_model_right" value="$(arg wrist_model_right)" />
-    <xacro:property name="has_arm_left" value="${arm_left != 'no-arm'}"/>
-    <xacro:property name="has_arm_right" value="${arm_right != 'no-arm'}"/>
-    <xacro:property name="end_effector_left" value="$(arg end_effector_left)" />
-    <xacro:property name="end_effector_right" value="$(arg end_effector_right)" />
-    <xacro:property name="ft_sensor_left" value="$(arg ft_sensor_left)" />
-    <xacro:property name="ft_sensor_right" value="$(arg ft_sensor_right)" />
-    <xacro:property name="laser_model" value="$(arg laser_model)" />
-    <xacro:property name="camera_model" value="$(arg camera_model)" />
-    <xacro:property name="has_screen" value="$(arg has_screen)" />
-    <xacro:property name="base_type" value="$(arg base_type)" />
-    <xacro:property name="is_multiple" value="$(arg multiple)" />
-    <xacro:property name="nsp" value="$(arg namespace)" />
-    <xacro:property name="no_safety_eps" value="$(arg no_safety_eps)" />
+<robot xmlns:xacro="http://ros.org/wiki/xacro" name="tiago_dual">
+  <!-- ARGUMENTS -->
+  <!-- tiago-arm, no-arm -->
+  <xacro:arg name="arm_left" default="tiago-arm"/>
+  <!-- tiago-arm, no-arm -->
+  <xacro:arg name="arm_right" default="tiago-arm"/>
+  <xacro:arg name="wrist_model_left" default="wrist-2010"/>
+  <xacro:arg name="wrist_model_right" default="wrist-2010"/>
+  <!-- no-end-effector, pal-gripper, pal-hey5, custom-->
+  <xacro:arg name="end_effector_left" default="pal-gripper"/>
+  <!-- no-end-effector, pal-gripper, pal-hey5, custom-->
+  <xacro:arg name="end_effector_right" default="pal-gripper"/>
+  <!--no-ft-sensor, schunk-ft -->
+  <xacro:arg name="ft_sensor_left" default="schunk-ft"/>
+  <!--no-ft-sensor, schunk-ft -->
+  <xacro:arg name="ft_sensor_right" default="schunk-ft"/>
+  <!-- no-laser, hokuyo, sick-551, sick-561, sick-571-->
+  <xacro:arg name="laser_model" default="sick-571"/>
+  <!-- no-camera, orbbec-astra, orbbec-astra-pro, asus-xtion -->
+  <xacro:arg name="camera_model" default="orbbec-astra"/>
+  <!-- pmb2, omni_base -->
+  <xacro:arg name="base_type" default="pmb2"/>
+  <xacro:arg name="description_calibration_dir" default="$(find tiago_dual_description)/urdf/calibration"/>
+  <xacro:arg name="extrinsic_calibration_dir" default="$(find tiago_dual_description)/urdf/calibration"/>
+  <xacro:arg name="namespace" default=""/>
+  <xacro:arg name="no_safety_eps" default="false"/>
+  <xacro:arg name="use_sim" default="false"/>
+  <xacro:arg name="has_screen" default="false"/>
+  <xacro:arg name="multiple" default="false"/>
+  <!-- PROPERTIES -->
+  <xacro:property name="arm_left" value="$(arg arm_left)"/>
+  <xacro:property name="arm_right" value="$(arg arm_right)"/>
+  <xacro:property name="wrist_model_left" value="$(arg wrist_model_left)" />
+  <xacro:property name="wrist_model_right" value="$(arg wrist_model_right)" />
+  <xacro:property name="end_effector_left" value="$(arg end_effector_left)" />
+  <xacro:property name="end_effector_right" value="$(arg end_effector_right)" />
+  <xacro:property name="ft_sensor_left" value="$(arg ft_sensor_left)" />
+  <xacro:property name="ft_sensor_right" value="$(arg ft_sensor_right)" />
+  <xacro:property name="laser_model" value="$(arg laser_model)" />
+  <xacro:property name="camera_model" value="$(arg camera_model)" />
+  <xacro:property name="has_screen" value="$(arg has_screen)" />
+  <xacro:property name="base_type" value="$(arg base_type)" />
+  <xacro:property name="is_multiple" value="$(arg multiple)" />
+  <xacro:property name="nsp" value="$(arg namespace)" />
+  <xacro:property name="no_safety_eps" value="$(arg no_safety_eps)" />
+  <xacro:property name="head_link_name" value="head_2_link"/>
+  <xacro:property name="description_calibration_dir" value="${arg description_calibration_dir}"/>
+  <xacro:property name="has_arm_left" value="${arm_left != 'no-arm'}"/>
+  <xacro:property name="has_ft_sensor_left" value="${ft_sensor_left != 'no-ft-sensor'}"/>
+  <xacro:property name="has_end_effector_left" value="${end_effector_left not in ['false', 'False', 'no-ee']}"/>
+  <xacro:property name="end_effector_left_link" value="${'wrist_left_ft_tool_link' if has_ft_sensor_left else 'arm_left_tool_link'}"/>
+  <xacro:property name="end_effector_left_name" value="${'hand_left' if end_effector_left == 'pal-hey5' else 'gripper_left'}"/>
+  <xacro:property name="has_arm_right" value="${arm_right != 'no-arm'}"/>
+  <xacro:property name="has_ft_sensor_right" value="${ft_sensor_right != 'no-ft-sensor'}"/>
+  <xacro:property name="has_end_effector_right" value="${end_effector_right not in ['false', 'False', 'no-ee']}"/>
+  <xacro:property name="end_effector_right_link" value="${'wrist_right_ft_tool_link' if has_ft_sensor_right else 'arm_right_tool_link'}"/>
+  <xacro:property name="end_effector_right_name" value="${'hand_right' if end_effector_right == 'pal-hey5' else 'gripper_right'}"/>
+  <!-- Properties check -->
   <xacro:if value="${arm_left not in ['no-arm', 'tiago-arm']}">
     <xacro:wrong_arm_left_type/>
@@ -82,16 +103,6 @@
     <xacro:wrong_base_type/>
   </xacro:if>
-   <xacro:property name="has_ft_sensor_left"      value="${ft_sensor_left != 'no-ft-sensor'}"/> <!-- This should be OR'ed with other FT sensors-->
-   <xacro:property name="has_ft_sensor_right"     value="${ft_sensor_right != 'no-ft-sensor'}"/> <!-- This should be OR'ed with other FT sensors-->
-   <xacro:property name="has_end_effector_left"        value="${end_effector_left not in ['false', 'False', 'no-ee']}"/>
-   <xacro:property name="end_effector_left_link"       value="${'wrist_left_ft_tool_link' if has_ft_sensor_left else 'arm_left_tool_link'}"/>
-   <xacro:property name="end_effector_left_name"       value="${'hand_left' if end_effector_left == 'pal-hey5' else 'gripper_left'}"/>
-   <xacro:property name="has_end_effector_right"        value="${end_effector_right not in ['false', 'False', 'no-ee']}"/>
-   <xacro:property name="end_effector_right_link"       value="${'wrist_right_ft_tool_link' if has_ft_sensor_right else 'arm_right_tool_link'}"/>
-   <xacro:property name="end_effector_right_name"       value="${'hand_right' if end_effector_right == 'pal-hey5' else 'gripper_right'}"/>
-   <xacro:property name="head_link_name"          value="head_2_link"/>
-   <xacro:property name="description_calibration_dir"       value="${arg description_calibration_dir}"/>
-  <!-- The following included files set up definitions of parts of the robot body -->
-  <!--File includes-->
+  <!-- INCLUDES -->
+  <!-- Tools -->
   <xacro:include filename="$(find pal_urdf_utils)/urdf/deg_to_rad.urdf.xacro" />
   <!-- Base -->
@@ -99,12 +110,19 @@
   <!-- Torso -->
   <xacro:include filename="$(find tiago_dual_description)/urdf/torso/torso_dual.urdf.xacro" />
+  <!-- Calibration constants -->
+  <xacro:include filename="$(arg description_calibration_dir)/calibration_constants.urdf.xacro" />
   <!-- Arm -->
-  <xacro:include filename="$(arg description_calibration_dir)/calibration_constants.urdf.xacro" />
-  <xacro:include filename="$(find tiago_description)/urdf/arm/arm.urdf.xacro" />
+  <xacro:if value="${has_arm_right or has_arm_left}">
+    <xacro:include filename="$(find tiago_description)/urdf/arm/arm.urdf.xacro" />
+  </xacro:if>
   <!-- End Effector -->
-  <xacro:include filename="$(find tiago_description)/urdf/end_effector/end_effector.urdf.xacro" />
+  <xacro:if value="${(has_arm_right or has_arm_left) and (has_end_effector_right or has_end_effector_left)}">
+    <xacro:include filename="$(find tiago_description)/urdf/end_effector/end_effector.urdf.xacro" />
+  </xacro:if>
   <!-- Force Torque sensor -->
-  <xacro:include filename="$(find tiago_description)/urdf/sensors/ftsensor.urdf.xacro" />
-  <xacro:include filename="$(find tiago_description)/urdf/sensors/ftsensor.gazebo.xacro" />
+  <xacro:if value="${(has_arm_right or has_arm_left) and (has_ft_sensor_right or has_ft_sensor_left)}">
+    <xacro:include filename="$(find tiago_description)/urdf/sensors/ftsensor.urdf.xacro" />
+    <xacro:include filename="$(find tiago_description)/urdf/sensors/ftsensor.gazebo.xacro" />
+  </xacro:if>
   <!-- Head -->
   <xacro:include filename="$(find tiago_description)/urdf/head/head.urdf.xacro" />
@@ -113,9 +131,8 @@
   <!-- Generic simulator_gazebo plugins -->
   <xacro:include filename="$(find tiago_description)/gazebo/gazebo.urdf.xacro" />
-  <!-- ros2_control -->
+  <!-- ROS 2 Control -->
   <xacro:include filename="$(find tiago_dual_description)/ros2_control/ros2_control.urdf.xacro" />
-  <xacro:tiago_dual_ros2_control
-    use_sim="$(arg use_sim)" />
-  <!-- Now we can start using the macros included above to define the actual robot -->
+  <!-- ROBOT DEFINITION -->
+  <!-- Base -->
   <xacro:if value="${base_type == 'pmb2'}">
     <xacro:base_sensors name="base" laser_model="$(arg laser_model)" sonars="true" microphone="true"/>
@@ -124,43 +141,53 @@
     <xacro:base_sensors name="base" front_laser_model="$(arg laser_model)" rear_laser_model="$(arg laser_model)"/>
   </xacro:if> -->
+  <!-- Torso -->
   <xacro:tiago_dual_torso name="torso" parent="base_link" has_screen="$(arg has_screen)"/>
-  <xacro:head name="head" parent="torso_lift_link" camera_model="$(arg camera_model)"
-	  description_calibration_dir="$(arg description_calibration_dir)"
-	  extrinsic_calibration_dir="$(arg extrinsic_calibration_dir)"
-    no_safety_eps="${no_safety_eps}"/>
-  <!-- Left -->
+  <!-- Head -->
+  <xacro:head name="head" parent="torso_lift_link" camera_model="$(arg camera_model)" description_calibration_dir="$(arg description_calibration_dir)" extrinsic_calibration_dir="$(arg extrinsic_calibration_dir)" no_safety_eps="${no_safety_eps}"/>
+  <!-- Left arm -->
   <xacro:if value="${has_arm_left}">
-	  <xacro:tiago_arm name="arm_left" parent="torso_lift_link" wrist_model="${wrist_model_left}" has_ft_sensor="${has_ft_sensor_left}" reflect="-1" tiago_dual="1" arm_1_offset="${arm_left_1_joint_offset}" arm_2_offset="${arm_left_2_joint_offset}" arm_3_offset="${arm_left_3_joint_offset}" arm_4_offset="${arm_left_4_joint_offset}" arm_5_offset="${arm_left_5_joint_offset}" arm_6_offset="${arm_left_6_joint_offset}" arm_7_offset="${arm_left_7_joint_offset}" no_safety_eps="${no_safety_eps}">
-	    <origin xyz="0.02556 0.19 -0.171" rpy="${180 * deg_to_rad} 0 ${90 * deg_to_rad}"/>
-	  </xacro:tiago_arm>
-	  <xacro:if value="${has_ft_sensor_left}">
-	      <xacro:ft_sensor name="wrist_left" parent="arm_left_tool_link" />
-        <xacro:force_torque_sensor_gazebo name="wrist_left_ft" update_rate="100"/>
-	  </xacro:if>
-  <xacro:tiago_end_effector name="${end_effector_left_name}" parent="${end_effector_left_link}" type="${end_effector_left}" reflect="-1" tiago_dual="true"/>
+    <!-- Arm -->
+    <xacro:tiago_arm name="arm_left" parent="torso_lift_link" wrist_model="${wrist_model_left}" has_ft_sensor="${has_ft_sensor_left}" reflect="-1" tiago_dual="1" arm_1_offset="${arm_left_1_joint_offset}" arm_2_offset="${arm_left_2_joint_offset}" arm_3_offset="${arm_left_3_joint_offset}" arm_4_offset="${arm_left_4_joint_offset}" arm_5_offset="${arm_left_5_joint_offset}" arm_6_offset="${arm_left_6_joint_offset}" arm_7_offset="${arm_left_7_joint_offset}" no_safety_eps="${no_safety_eps}">
+      <origin xyz="0.02556 0.19 -0.171" rpy="${180 * deg_to_rad} 0 ${90 * deg_to_rad}"/>
+    </xacro:tiago_arm>
+    <!-- End effector -->
+    <xacro:if value="${has_end_effector_left}">
+      <xacro:tiago_end_effector name="${end_effector_left_name}" parent="${end_effector_left_link}" type="${end_effector_left}" reflect="-1" tiago_dual="true"/>
+    </xacro:if>
+    <!-- FT sensors -->
+    <xacro:if value="${has_ft_sensor_left}">
+      <xacro:ft_sensor name="wrist_left" parent="arm_left_tool_link" />
+      <xacro:force_torque_sensor_gazebo name="wrist_left_ft" update_rate="100"/>
+    </xacro:if>
   </xacro:if>
-  <!-- Right -->
+  <!-- Right arm -->
   <xacro:if value="${has_arm_right}">
-	  <xacro:tiago_arm name="arm_right" parent="torso_lift_link" wrist_model="${wrist_model_right}" has_ft_sensor="${has_ft_sensor_right}" reflect="1" tiago_dual="1" arm_1_offset="${arm_right_1_joint_offset}" arm_2_offset="${arm_right_2_joint_offset}" arm_3_offset="${arm_right_3_joint_offset}" arm_4_offset="${arm_right_4_joint_offset}" arm_5_offset="${arm_right_5_joint_offset}" arm_6_offset="${arm_right_6_joint_offset}" arm_7_offset="${arm_right_7_joint_offset}"  no_safety_eps="${no_safety_eps}">
-	    <origin xyz="0.02556 -0.19 -0.171" rpy="0 0 ${-90 * deg_to_rad}"/>
-	  </xacro:tiago_arm>
-	  <xacro:if value="${has_ft_sensor_right}">
-	      <xacro:ft_sensor name="wrist_right" parent="arm_right_tool_link" />
-        <xacro:force_torque_sensor_gazebo name="wrist_right_ft" update_rate="100"/>
-	  </xacro:if>
-	  <xacro:tiago_end_effector name="${end_effector_right_name}" parent="${end_effector_right_link}" type="${end_effector_right}" reflect="1" tiago_dual="true"/>
+    <!-- Arm -->
+    <xacro:tiago_arm name="arm_right" parent="torso_lift_link" wrist_model="${wrist_model_right}" has_ft_sensor="${has_ft_sensor_right}" reflect="1" tiago_dual="1" arm_1_offset="${arm_right_1_joint_offset}" arm_2_offset="${arm_right_2_joint_offset}" arm_3_offset="${arm_right_3_joint_offset}" arm_4_offset="${arm_right_4_joint_offset}" arm_5_offset="${arm_right_5_joint_offset}" arm_6_offset="${arm_right_6_joint_offset}" arm_7_offset="${arm_right_7_joint_offset}" no_safety_eps="${no_safety_eps}">
+      <origin xyz="0.02556 -0.19 -0.171" rpy="0 0 ${-90 * deg_to_rad}"/>
+    </xacro:tiago_arm>
+    <xacro:if value="${has_ft_sensor_right}">
+      <xacro:ft_sensor name="wrist_right" parent="arm_right_tool_link" />
+      <xacro:force_torque_sensor_gazebo name="wrist_right_ft" update_rate="100"/>
+    </xacro:if>
+    <!-- End effector -->
+    <xacro:if value="${has_end_effector_right}">
+      <xacro:tiago_end_effector name="${end_effector_right_name}" parent="${end_effector_right_link}" type="${end_effector_right}" reflect="1" tiago_dual="true"/>
+    </xacro:if>
   </xacro:if>
+  <!-- ROS 2 Control -->
+  <xacro:tiago_dual_ros2_control use_sim="$(arg use_sim)" />
   <!-- RGBD Laser Link -->
   <joint name="rgbd_laser_joint" type="fixed">
-      <parent link="base_footprint"/>
-      <child link="rgbd_laser_link"/>
-      <origin xyz="-0.9 0 0" rpy="0 0 0" />
+    <parent link="base_footprint"/>
+    <child link="rgbd_laser_link"/>
+    <origin xyz="-0.9 0 0" rpy="0 0 0" />
   </joint>
   <link name="rgbd_laser_link">
-      <inertial>
-          <origin xyz="0 0 0" rpy="0 0 0"/>
-          <mass value="0.0001" />
-          <inertia ixx="0.0001"  ixy="0"  ixz="0" iyy="0.0001" iyz="0" izz="0.0001" />
-      </inertial>
+    <inertial>
+      <origin xyz="0 0 0" rpy="0 0 0"/>
+      <mass value="0.0001" />
+      <inertia ixx="0.0001" ixy="0" ixz="0" iyy="0.0001" iyz="0" izz="0.0001" />
+    </inertial>
   </link>
 </robot>
